Commit message: creating planner class

File: pursuit3d/urdf/campus.urdf (robot description, URDF)
Before this commit: robot test_robot, 4 links, 3 joints
Links:
- removed link link1
- removed link link2
- removed link link3
- removed link link4
- added link chem; collision box size=8 8 29.9
- added link inertial
- added link meem; collision box size=10 10 40.8
Joints:
- removed joint joint1
- removed joint joint2
- removed joint joint3
- added joint joint_chem: type fixed, parent inertial, child chem
- added joint joint_meem: type fixed, parent inertial, child meem
